Commit message: Add files via upload

File: src/urdf01_rviz/urdf/xacro/demo05_car_base.urdf.xacro (robot description, xacro)
@@ -4,14 +4,7 @@
     <!-- 宏:黑色设置 -->
     <xacro:property name="footprint_radius" value="0.001" /> <!-- base_footprint 半径  -->
-<!--
     <material name="black">
         <color rgba="0.0 0.0 0.0 1.0" />
-    </material> -->
-    <!-- 底盘属性 -->
-    <xacro:property name="base_radius" value="0.1" /> <!-- base_link 半径 -->
-    <xacro:property name="base_length" value="0.08" /> <!-- base_link 长 -->
-    <xacro:property name="lidi" value="0.015" /> <!-- 离地间距 -->
-    <xacro:property name="base_joint_z" value="${base_length /2 + lidi}" /> <!-- 离地间距 -->
-    <!-- 底盘 -->
+    </material>
     <link name="base_footprint">
       <visual>
@@ -21,4 +14,15 @@
       </visual>
     </link>
+    <!-- 底盘属性
+    形狀：cylinder
+    半徑：0.1m
+    高度：0.08m
+    離地間距：0.015m    -->
+    <xacro:property name="base_radius" value="0.1" /> <!-- base_link 半径 -->
+    <xacro:property name="base_length" value="0.08" /> <!-- base_link 长 -->
+    <xacro:property name="lidi" value="0.015" /> <!-- 离地间距 -->
+    <xacro:property name="base_joint_z" value="${base_length /2 + lidi}" /> <!-- 离地间距 -->
+    <xacro:property name="base_mass" value="0.5" /> <!-- 质量  -->
+    <!-- 底盘link -->
     <link name="base_link">
       <visual>
@@ -27,9 +31,20 @@
         </geometry>
         <origin xyz="0 0 0" rpy="0 0 0" />
-        <material name="yellow">
-          <color rgba="0.5 0.3 0.0 0.5" />
+        <material name="base_link_color">
+          <color rgba="1.0 0.5 0.2 0.5" />
         </material>
       </visual>
+      <collision>     <!-- 底盤碰撞 -->
+          <geometry>
+            <cylinder radius="${base_radius}" length="${base_length}" />
+          </geometry>
+          <origin xyz="0 0 0" rpy="0 0 0" />
+      </collision>
+      <!-- 調用慣性 -->
+      <xacro:cylinder_inertial_matrix m="${base_mass}" r="${base_radius}" h="${base_length}" />
     </link>
+    <gazebo reference="base_link">
+        <material>Gazebo/Yellow</material> <!-- 設置gazebo顔色 -->
+    </gazebo>
     <joint name="link2footprint" type="fixed">
       <parent link="base_footprint" />
@@ -37,5 +52,5 @@
       <origin xyz="0 0 0.055" rpy= "0 0 0"/>
     </joint>
-    <!-- 驱动轮 -->
+    <!-- 驱动轮1111111111111111111111111111111111111111111111111111111111111111 -->
     <!-- 驱动轮属性 -->
     <xacro:property name="wheel_radius" value="0.0325" /><!-- 半径 -->
@@ -43,4 +58,5 @@
     <xacro:property name="PI" value="3.1415"/>
     <xacro:property name="wheel_joint_z" value="${(base_length / 2 + lidi - wheel_radius)*-1}" /> <!-- 离地间距 -->
+    <xacro:property name="wheel_mass" value="0.05" /> <!-- 质量  -->
     <!-- 驱动轮宏实现 -->
     <xacro:macro name="wheels_func" params="wheel_name flag">
@@ -53,5 +69,16 @@
           <material name="black" />
         </visual>
+        <collision> <!-- 驅動輪碰撞 -->
+          <geometry>
+            <cylinder radius="${wheel_radius}" length="${wheel_length}" />
+          </geometry>
+          <origin xyz="0.0 0.0 0.0" rpy="${PI / 2} 0.0 0.0" />
+        </collision>
+      <!-- 調用慣性 -->
+        <xacro:cylinder_inertial_matrix m="${wheel_mass}" r="${wheel_radius}" h="${wheel_length}" />
       </link>
+      <gazebo reference="${wheel_name}_wheel">
+        <material>Gazebo/Red</material>  <!-- 設置gazebo顔色 -->
+      </gazebo>
       <joint name="${wheel_name}2link" type="continuous">
         <parent link="base_link" />
@@ -63,9 +90,10 @@
     <xacro:wheels_func wheel_name="left" flag="1" />
     <xacro:wheels_func wheel_name="right" flag="-1" />
-    <!-- 支撑轮 -->
+    <!-- 支撑轮11111111111111111111111111111111111111111111111111111111111111 -->
     <!-- 支撑轮属性 -->
     <!-- z 的偏移量 = 車輪高度 /2 + 離地間距 - 萬向輪半徑 -->
     <xacro:property name="small_wheel_radius" value="0.0075" /> <!-- 支撑轮半径 -->
     <xacro:property name="small_joint_z" value="${(base_length / 2 + lidi - small_wheel_radius)*-1}" /> <!-- 离地间距 -->
+    <xacro:property name="support_wheel_m" value="0.03" /> <!-- 质量  -->
     <!-- 支撑轮宏 -->
     <xacro:macro name="small_wheel_func" params="small_wheel_name flag" >
@@ -78,4 +106,12 @@
             <material name="black" />
         </visual>
+        <collision> <!-- 支撐輪碰撞 -->
+            <geometry>
+                <sphere radius="${small_wheel_radius}" />
+            </geometry>
+            <origin xyz="0 0 0" rpy="0 0 0" />
+        </collision>
+      <!-- 調用慣性 -->
+        <xacro:sphere_inertial_matrix m="${support_wheel_m}" r="${small_wheel_radius}" />
       </link>
       <joint name="${small_wheel_name}2link" type="continuous">
@@ -85,4 +121,7 @@
           <axis xyz="1 1 1" />
       </joint>
+      <gazebo reference="${small_wheel_name}_wheel"> <!-- 設置gazebo顔色 -->
+        <material>Gazebo/Red</material>
+      </gazebo>
     </xacro:macro>
     <xacro:small_wheel_func small_wheel_name="front" flag="1" />

File: src/urdf01_rviz/urdf/xacro/demo06_car_camera.urdf.xacro (robot description, xacro)
@@ -8,4 +8,5 @@
     <xacro:property name="joint_camera_y" value="0.0" /> <!-- 摄像头安装的y坐标 -->
     <xacro:property name="joint_camera_z" value="${base_length / 2 + camera_height / 2}" /> <!-- 摄像头安装的z坐标:底盘高度 / 2 + 摄像头高度 / 2  -->
+    <xacro:property name="camera_m" value="0.01" /> <!-- 摄像头质量=0.01kg-->
     <!-- 摄像头关节以及link -->
     <link name="camera">
@@ -16,4 +17,12 @@
             <material name="black" />
         </visual>
+        <collision>       <!-- 鏡頭碰撞 -->
+            <geometry>
+                <box size="${camera_length} ${camera_width} ${camera_height}" />
+            </geometry>
+            <origin xyz="0.0 0.0 0.0" rpy="0.0 0.0 0.0" />
+        </collision>
+      <!-- 調用慣性 -->
+        <xacro:Box_inertial_matrix m="${camera_m}" l="${camera_length}" w="${camera_width}" h="${camera_height}" />
     </link>
     <joint name="camera2base" type="fixed">
@@ -22,3 +31,6 @@
         <origin xyz="${joint_camera_x} ${joint_camera_y} ${joint_camera_z}" />
     </joint>
+    <gazebo reference="camera">
+        <material>Gazebo/Blue</material> <!-- 設置gazebo顔色 -->
+    </gazebo>
 </robot>

File: src/urdf01_rviz/urdf/xacro/demo07_car_laser.urdf.xacro (robot description, xacro)
@@ -14,4 +14,6 @@
     <xacro:property name="joint_laser_y" value="0.0" /> <!-- 雷达安装的y坐标 -->
     <xacro:property name="joint_laser_z" value="${support_length / 2 + laser_length / 2}" /> <!-- 雷达安装的z坐标:支架高度 / 2 + 雷达高度 / 2  -->
+    <xacro:property name="support_m" value="0.02" /> <!-- 支架质量 -->
+    <xacro:property name="laser_m" value="0.1" /> <!-- 雷达质量 -->
     <link name="support">
         <visual>
@@ -24,4 +26,12 @@
             </material>
         </visual>
+        <collision> <!-- 碰撞 -->
+            <geometry>
+                <cylinder radius="${support_radius}" length="${support_length}" />
+            </geometry>
+            <origin xyz="0.0 0.0 0.0" rpy="0.0 0.0 0.0" />
+        </collision>
+      <!-- 調用慣性 -->
+        <xacro:cylinder_inertial_matrix m="${support_m}" r="${support_radius}" h="${support_length}" />
     </link>
     <joint name="support2base" type="fixed">
@@ -30,4 +40,7 @@
         <origin xyz="${joint_support_x} ${joint_support_y} ${joint_support_z}" />
     </joint>
+    <gazebo reference="support">
+        <material>Gazebo/White</material>
+    </gazebo>
     <!-- 雷达关节以及link -->
     <link name="laser">
@@ -39,5 +52,16 @@
             <material name="black" />
         </visual>
+        <collision> <!--碰撞 -->
+            <geometry>
+                <cylinder radius="${laser_radius}" length="${laser_length}" />
+            </geometry>
+            <origin xyz="0.0 0.0 0.0" rpy="0.0 0.0 0.0" />
+        </collision>
+      <!-- 調用慣性 -->
+        <xacro:cylinder_inertial_matrix m="${laser_m}" r="${laser_radius}" h="${laser_length}" />
     </link>
+    <gazebo reference="laser">
+        <material>Gazebo/Black</material>
+    </gazebo>
     <joint name="laser2support" type="fixed">
         <parent link="support" />

File: urdf02_gazebo/urdf/demo05_car_base.urdf.xacro (robot description, xacro)
@@ -1,66 +1,65 @@
-<!--
-    使用 xacro 优化 URDF 版的小车底盘实现：
-    实现思路:
-    1.将一些常量、变量封装为 xacro:property
-      比如:PI 值、小车底盘半径、离地间距、车轮半径、宽度 ....
-    2.使用 宏 封装驱动轮以及支撑轮实现，调用相关宏生成驱动轮与支撑轮
--->
 <!-- 根标签，必须声明 xmlns:xacro -->
 <robot name="my_base" xmlns:xacro="http://www.ros.org/wiki/xacro">
     <!-- 封装变量、常量 -->
-    <!-- PI 值设置精度需要高一些，否则后续车轮翻转量计算时，可能会出现肉眼不能察觉的车轮倾斜，从而导致模型抖动 -->
-    <xacro:property name="PI" value="3.1415926"/>
     <!-- 宏:黑色设置 -->
+    <xacro:property name="footprint_radius" value="0.001" /> <!-- base_footprint 半径  -->
     <material name="black">
         <color rgba="0.0 0.0 0.0 1.0" />
     </material>
-    <!-- 底盘属性 -->
-    <xacro:property name="base_footprint_radius" value="0.001" /> <!-- base_footprint 半径  -->
-    <xacro:property name="base_link_radius" value="0.1" /> <!-- base_link 半径 -->
-    <xacro:property name="base_link_length" value="0.08" /> <!-- base_link 长 -->
-    <xacro:property name="earth_space" value="0.015" /> <!-- 离地间距 -->
-    <xacro:property name="base_link_m" value="0.5" /> <!-- 质量  -->
-    <!-- 底盘 -->
     <link name="base_footprint">
       <visual>
         <geometry>
-          <sphere radius="${base_footprint_radius}" />
+          <sphere radius="${footprint_radius}" />
         </geometry>
       </visual>
     </link>
+    <!-- 底盘属性
+    形狀：cylinder
+    半徑：0.1m
+    高度：0.08m
+    離地間距：0.015m    -->
+    <xacro:property name="base_radius" value="0.1" /> <!-- base_link 半径 -->
+    <xacro:property name="base_length" value="0.08" /> <!-- base_link 长 -->
+    <xacro:property name="lidi" value="0.015" /> <!-- 离地间距 -->
+    <xacro:property name="base_joint_z" value="${base_length /2 + lidi}" /> <!-- 离地间距 -->
+    <xacro:property name="base_mass" value="0.5" /> <!-- 质量  -->
+    <!-- 底盘link -->
     <link name="base_link">
       <visual>
         <geometry>
-          <cylinder radius="${base_link_radius}" length="${base_link_length}" />
+          <cylinder radius="${base_radius}" length="${base_length}" />
         </geometry>
         <origin xyz="0 0 0" rpy="0 0 0" />
-        <material name="yellow">
-          <color rgba="0.5 0.3 0.0 0.5" />
+        <material name="base_link_color">
+          <color rgba="1.0 0.5 0.2 0.5" />
         </material>
       </visual>
-      <collision>
-        <geometry>
-          <cylinder radius="${base_link_radius}" length="${base_link_length}" />
-        </geometry>
-        <origin xyz="0 0 0" rpy="0 0 0" />
+      <collision>     <!-- 底盤碰撞 -->
+          <geometry>
+            <cylinder radius="${base_radius}" length="${base_length}" />
+          </geometry>
+          <origin xyz="0 0 0" rpy="0 0 0" />
       </collision>
-      <xacro:cylinder_inertial_matrix m="${base_link_m}" r="${base_link_radius}" h="${base_link_length}" />
+      <!-- 調用慣性 -->
+      <xacro:cylinder_inertial_matrix m="${base_mass}" r="${base_radius}" h="${base_length}" />
     </link>
-    <joint name="base_link2base_footprint" type="fixed">
+    <gazebo reference="base_link">
+        <material>Gazebo/Yellow</material> <!-- 設置gazebo顔色 -->
+    </gazebo>
+    <joint name="link2footprint" type="fixed">
       <parent link="base_footprint" />
       <child link="base_link" />
-      <origin xyz="0 0 ${earth_space + base_link_length / 2 }" />
+      <origin xyz="0 0 0.055" rpy= "0 0 0"/>
     </joint>
-    <gazebo reference="base_link">
-        <material>Gazebo/Yellow</material>
-    </gazebo>
-    <!-- 驱动轮 -->
+    <!-- 驱动轮1111111111111111111111111111111111111111111111111111111111111111 -->
     <!-- 驱动轮属性 -->
     <xacro:property name="wheel_radius" value="0.0325" /><!-- 半径 -->
     <xacro:property name="wheel_length" value="0.015" /><!-- 宽度 -->
-    <xacro:property name="wheel_m" value="0.05" /> <!-- 质量  -->
+    <xacro:property name="PI" value="3.1415"/>
+    <xacro:property name="wheel_joint_z" value="${(base_length / 2 + lidi - wheel_radius)*-1}" /> <!-- 离地间距 -->
+    <xacro:property name="wheel_mass" value="0.05" /> <!-- 质量  -->
     <!-- 驱动轮宏实现 -->
-    <xacro:macro name="add_wheels" params="name flag">
-      <link name="${name}_wheel">
+    <xacro:macro name="wheels_func" params="wheel_name flag">
+      <link name="${wheel_name}_wheel">
         <visual>
           <geometry>
@@ -70,5 +69,5 @@
           <material name="black" />
         </visual>
-        <collision>
+        <collision> <!-- 驅動輪碰撞 -->
           <geometry>
             <cylinder radius="${wheel_radius}" length="${wheel_length}" />
@@ -76,51 +75,55 @@
           <origin xyz="0.0 0.0 0.0" rpy="${PI / 2} 0.0 0.0" />
         </collision>
-        <xacro:cylinder_inertial_matrix m="${wheel_m}" r="${wheel_radius}" h="${wheel_length}" />
+      <!-- 調用慣性 -->
+        <xacro:cylinder_inertial_matrix m="${wheel_mass}" r="${wheel_radius}" h="${wheel_length}" />
       </link>
-      <joint name="${name}_wheel2base_link" type="continuous">
+      <gazebo reference="${wheel_name}_wheel">
+        <material>Gazebo/Red</material>  <!-- 設置gazebo顔色 -->
+      </gazebo>
+      <joint name="${wheel_name}2link" type="continuous">
         <parent link="base_link" />
-        <child link="${name}_wheel" />
-        <origin xyz="0 ${flag * base_link_radius} ${-(earth_space + base_link_length / 2 - wheel_radius) }" />
+        <child link="${wheel_name}_wheel" />
+        <origin xyz="0 ${0.1 * flag} ${wheel_joint_z} " rpy="0.0 0.0 0.0" />
         <axis xyz="0 1 0" />
       </joint>
-      <gazebo reference="${name}_wheel">
-        <material>Gazebo/Red</material>
-      </gazebo>
     </xacro:macro>
-    <xacro:add_wheels name="left" flag="1" />
-    <xacro:add_wheels name="right" flag="-1" />
-    <!-- 支撑轮 -->
+    <xacro:wheels_func wheel_name="left" flag="1" />
+    <xacro:wheels_func wheel_name="right" flag="-1" />
+    <!-- 支撑轮11111111111111111111111111111111111111111111111111111111111111 -->
     <!-- 支撑轮属性 -->
-    <xacro:property name="support_wheel_radius" value="0.0075" /> <!-- 支撑轮半径 -->
+    <!-- z 的偏移量 = 車輪高度 /2 + 離地間距 - 萬向輪半徑 -->
+    <xacro:property name="small_wheel_radius" value="0.0075" /> <!-- 支撑轮半径 -->
+    <xacro:property name="small_joint_z" value="${(base_length / 2 + lidi - small_wheel_radius)*-1}" /> <!-- 离地间距 -->
     <xacro:property name="support_wheel_m" value="0.03" /> <!-- 质量  -->
     <!-- 支撑轮宏 -->
-    <xacro:macro name="add_support_wheel" params="name flag" >
-      <link name="${name}_wheel">
+    <xacro:macro name="small_wheel_func" params="small_wheel_name flag" >
+      <link name="${small_wheel_name}_wheel">
         <visual>
             <geometry>
-                <sphere radius="${support_wheel_radius}" />
+                <sphere radius="${small_wheel_radius}" />
             </geometry>
             <origin xyz="0 0 0" rpy="0 0 0" />
             <material name="black" />
         </visual>
-        <collision>
+        <collision> <!-- 支撐輪碰撞 -->
             <geometry>
-                <sphere radius="${support_wheel_radius}" />
+                <sphere radius="${small_wheel_radius}" />
             </geometry>
             <origin xyz="0 0 0" rpy="0 0 0" />
         </collision>
-        <xacro:sphere_inertial_matrix m="${support_wheel_m}" r="${support_wheel_radius}" />
+      <!-- 調用慣性 -->
+        <xacro:sphere_inertial_matrix m="${support_wheel_m}" r="${small_wheel_radius}" />
       </link>
-      <joint name="${name}_wheel2base_link" type="continuous">
+      <joint name="${small_wheel_name}2link" type="continuous">
           <parent link="base_link" />
-          <child link="${name}_wheel" />
-          <origin xyz="${flag * (base_link_radius - support_wheel_radius)} 0 ${-(base_link_length / 2 + earth_space / 2)}" />
+          <child link="${small_wheel_name}_wheel" />
+          <origin xyz="${flag * 0.08} 0 ${small_joint_z}" />
           <axis xyz="1 1 1" />
       </joint>
-      <gazebo reference="${name}_wheel">
+      <gazebo reference="${small_wheel_name}_wheel"> <!-- 設置gazebo顔色 -->
         <material>Gazebo/Red</material>
       </gazebo>
     </xacro:macro>
-    <xacro:add_support_wheel name="front" flag="1" />
-    <xacro:add_support_wheel name="back" flag="-1" />
+    <xacro:small_wheel_func small_wheel_name="front" flag="1" />
+    <xacro:small_wheel_func small_wheel_name="back" flag="-1" />
 </robot>

File: urdf02_gazebo/urdf/demo06_car_camera.urdf.xacro (robot description, xacro)
@@ -2,11 +2,11 @@
 <robot name="my_camera" xmlns:xacro="http://wiki.ros.org/xacro">
     <!-- 摄像头属性 -->
-    <xacro:property name="camera_length" value="0.01" /> <!-- 摄像头长度(x) -->
-    <xacro:property name="camera_width" value="0.025" /> <!-- 摄像头宽度(y) -->
-    <xacro:property name="camera_height" value="0.025" /> <!-- 摄像头高度(z) -->
-    <xacro:property name="camera_x" value="0.08" /> <!-- 摄像头安装的x坐标 -->
-    <xacro:property name="camera_y" value="0.0" /> <!-- 摄像头安装的y坐标 -->
-    <xacro:property name="camera_z" value="${base_link_length / 2 + camera_height / 2}" /> <!-- 摄像头安装的z坐标:底盘高度 / 2 + 摄像头高度 / 2  -->
-    <xacro:property name="camera_m" value="0.01" /> <!-- 摄像头质量 -->
+    <xacro:property name="camera_length" value="0.02" /> <!-- 摄像头长度(x) -->
+    <xacro:property name="camera_width" value="0.05" /> <!-- 摄像头宽度(y) -->
+    <xacro:property name="camera_height" value="0.05" /> <!-- 摄像头高度(z) -->
+    <xacro:property name="joint_camera_x" value="0.08" /> <!-- 摄像头安装的x坐标 -->
+    <xacro:property name="joint_camera_y" value="0.0" /> <!-- 摄像头安装的y坐标 -->
+    <xacro:property name="joint_camera_z" value="${base_length / 2 + camera_height / 2}" /> <!-- 摄像头安装的z坐标:底盘高度 / 2 + 摄像头高度 / 2  -->
+    <xacro:property name="camera_m" value="0.01" /> <!-- 摄像头质量=0.01kg-->
     <!-- 摄像头关节以及link -->
     <link name="camera">
@@ -15,8 +15,7 @@
                 <box size="${camera_length} ${camera_width} ${camera_height}" />
             </geometry>
-            <origin xyz="0.0 0.0 0.0" rpy="0.0 0.0 0.0" />
             <material name="black" />
         </visual>
-        <collision>
+        <collision>       <!-- 鏡頭碰撞 -->
             <geometry>
                 <box size="${camera_length} ${camera_width} ${camera_height}" />
@@ -24,13 +23,14 @@
             <origin xyz="0.0 0.0 0.0" rpy="0.0 0.0 0.0" />
         </collision>
+      <!-- 調用慣性 -->
         <xacro:Box_inertial_matrix m="${camera_m}" l="${camera_length}" w="${camera_width}" h="${camera_height}" />
     </link>
-    <joint name="camera2base_link" type="fixed">
+    <joint name="camera2base" type="fixed">
         <parent link="base_link" />
         <child link="camera" />
-        <origin xyz="${camera_x} ${camera_y} ${camera_z}" />
+        <origin xyz="${joint_camera_x} ${joint_camera_y} ${joint_camera_z}" />
     </joint>
     <gazebo reference="camera">
-        <material>Gazebo/Blue</material>
+        <material>Gazebo/Blue</material> <!-- 設置gazebo顔色 -->
     </gazebo>
 </robot>
