Commit message: Add files via upload

File: urdf02_gazebo/urdf/demo07_car_laser.urdf.xacro (robot description, xacro)
@@ -6,8 +6,14 @@
     <xacro:property name="support_length" value="0.15" /> <!-- 支架长度 -->
     <xacro:property name="support_radius" value="0.01" /> <!-- 支架半径 -->
-    <xacro:property name="support_x" value="0.0" /> <!-- 支架安装的x坐标 -->
-    <xacro:property name="support_y" value="0.0" /> <!-- 支架安装的y坐标 -->
-    <xacro:property name="support_z" value="${base_link_length / 2 + support_length / 2}" /> <!-- 支架安装的z坐标:底盘高度 / 2 + 支架高度 / 2  -->
+    <xacro:property name="laser_length" value="0.05" /> <!-- 雷达长度 -->
+    <xacro:property name="laser_radius" value="0.03" /> <!-- 雷达半径 -->
+    <xacro:property name="joint_support_x" value="0.0" /> <!-- 支架安装的x坐标 -->
+    <xacro:property name="joint_support_y" value="0.0" /> <!-- 支架安装的y坐标 -->
+    <xacro:property name="joint_support_z" value="${base_length / 2 + support_length / 2}" /> <!-- 支架安装的z坐标:底盘高度 / 2 + 支架高度 / 2  -->
+    <xacro:property name="joint_laser_x" value="0.0" /> <!-- 雷达安装的x坐标 -->
+    <xacro:property name="joint_laser_y" value="0.0" /> <!-- 雷达安装的y坐标 -->
+    <xacro:property name="joint_laser_z" value="${support_length / 2 + laser_length / 2}" /> <!-- 雷达安装的z坐标:支架高度 / 2 + 雷达高度 / 2  -->
     <xacro:property name="support_m" value="0.02" /> <!-- 支架质量 -->
+    <xacro:property name="laser_m" value="0.1" /> <!-- 雷达质量 -->
     <link name="support">
         <visual>
@@ -20,5 +26,5 @@
             </material>
         </visual>
-        <collision>
+        <collision> <!-- 碰撞 -->
             <geometry>
                 <cylinder radius="${support_radius}" length="${support_length}" />
@@ -26,21 +32,15 @@
             <origin xyz="0.0 0.0 0.0" rpy="0.0 0.0 0.0" />
         </collision>
+      <!-- 調用慣性 -->
         <xacro:cylinder_inertial_matrix m="${support_m}" r="${support_radius}" h="${support_length}" />
     </link>
-    <joint name="support2base_link" type="fixed">
+    <joint name="support2base" type="fixed">
         <parent link="base_link" />
         <child link="support" />
-        <origin xyz="${support_x} ${support_y} ${support_z}" />
+        <origin xyz="${joint_support_x} ${joint_support_y} ${joint_support_z}" />
     </joint>
     <gazebo reference="support">
         <material>Gazebo/White</material>
     </gazebo>
-    <!-- 雷达属性 -->
-    <xacro:property name="laser_length" value="0.05" /> <!-- 雷达长度 -->
-    <xacro:property name="laser_radius" value="0.03" /> <!-- 雷达半径 -->
-    <xacro:property name="laser_x" value="0.0" /> <!-- 雷达安装的x坐标 -->
-    <xacro:property name="laser_y" value="0.0" /> <!-- 雷达安装的y坐标 -->
-    <xacro:property name="laser_z" value="${support_length / 2 + laser_length / 2}" /> <!-- 雷达安装的z坐标:支架高度 / 2 + 雷达高度 / 2  -->
-    <xacro:property name="laser_m" value="0.1" /> <!-- 雷达质量 -->
     <!-- 雷达关节以及link -->
     <link name="laser">
@@ -52,5 +52,5 @@
             <material name="black" />
         </visual>
-        <collision>
+        <collision> <!--碰撞 -->
             <geometry>
                 <cylinder radius="${laser_radius}" length="${laser_length}" />
@@ -58,82 +58,14 @@
             <origin xyz="0.0 0.0 0.0" rpy="0.0 0.0 0.0" />
         </collision>
+      <!-- 調用慣性 -->
         <xacro:cylinder_inertial_matrix m="${laser_m}" r="${laser_radius}" h="${laser_length}" />
     </link>
+    <gazebo reference="laser">
+        <material>Gazebo/Black</material>
+    </gazebo>
     <joint name="laser2support" type="fixed">
         <parent link="support" />
         <child link="laser" />
-        <origin xyz="${laser_x} ${laser_y} ${laser_z}" />
+        <origin xyz="${joint_laser_x} ${joint_laser_y} ${joint_laser_z}" />
     </joint>
-    <gazebo reference="laser">
-        <material>Gazebo/Black</material>
-    </gazebo>
-</robot><!--
-    小车底盘添加雷达
--->
-<robot name="my_laser" xmlns:xacro="http://wiki.ros.org/xacro">
-    <!-- 雷达支架 -->
-    <xacro:property name="support_length" value="0.15" /> <!-- 支架长度 -->
-    <xacro:property name="support_radius" value="0.01" /> <!-- 支架半径 -->
-    <xacro:property name="support_x" value="0.0" /> <!-- 支架安装的x坐标 -->
-    <xacro:property name="support_y" value="0.0" /> <!-- 支架安装的y坐标 -->
-    <xacro:property name="support_z" value="${base_link_length / 2 + support_length / 2}" /> <!-- 支架安装的z坐标:底盘高度 / 2 + 支架高度 / 2  -->
-    <xacro:property name="support_m" value="0.02" /> <!-- 支架质量 -->
-    <link name="support">
-        <visual>
-            <geometry>
-                <cylinder radius="${support_radius}" length="${support_length}" />
-            </geometry>
-            <origin xyz="0.0 0.0 0.0" rpy="0.0 0.0 0.0" />
-            <material name="red">
-                <color rgba="0.8 0.2 0.0 0.8" />
-            </material>
-        </visual>
-        <collision>
-            <geometry>
-                <cylinder radius="${support_radius}" length="${support_length}" />
-            </geometry>
-            <origin xyz="0.0 0.0 0.0" rpy="0.0 0.0 0.0" />
-        </collision>
-        <xacro:cylinder_inertial_matrix m="${support_m}" r="${support_radius}" h="${support_length}" />
-    </link>
-    <joint name="support2base_link" type="fixed">
-        <parent link="base_link" />
-        <child link="support" />
-        <origin xyz="${support_x} ${support_y} ${support_z}" />
-    </joint>
-    <gazebo reference="support">
-        <material>Gazebo/White</material>
-    </gazebo>
-    <!-- 雷达属性 -->
-    <xacro:property name="laser_length" value="0.05" /> <!-- 雷达长度 -->
-    <xacro:property name="laser_radius" value="0.03" /> <!-- 雷达半径 -->
-    <xacro:property name="laser_x" value="0.0" /> <!-- 雷达安装的x坐标 -->
-    <xacro:property name="laser_y" value="0.0" /> <!-- 雷达安装的y坐标 -->
-    <xacro:property name="laser_z" value="${support_length / 2 + laser_length / 2}" /> <!-- 雷达安装的z坐标:支架高度 / 2 + 雷达高度 / 2  -->
-    <xacro:property name="laser_m" value="0.1" /> <!-- 雷达质量 -->
-    <!-- 雷达关节以及link -->
-    <link name="laser">
-        <visual>
-            <geometry>
-                <cylinder radius="${laser_radius}" length="${laser_length}" />
-            </geometry>
-            <origin xyz="0.0 0.0 0.0" rpy="0.0 0.0 0.0" />
-            <material name="black" />
-        </visual>
-        <collision>
-            <geometry>
-                <cylinder radius="${laser_radius}" length="${laser_length}" />
-            </geometry>
-            <origin xyz="0.0 0.0 0.0" rpy="0.0 0.0 0.0" />
-        </collision>
-        <xacro:cylinder_inertial_matrix m="${laser_m}" r="${laser_radius}" h="${laser_length}" />
-    </link>
-    <joint name="laser2support" type="fixed">
-        <parent link="support" />
-        <child link="laser" />
-        <origin xyz="${laser_x} ${laser_y} ${laser_z}" />
-    </joint>
-    <gazebo reference="laser">
-        <material>Gazebo/Black</material>
-    </gazebo>
 </robot>
